File: hardware-design/kicad/dilder-breadboard/dilder-breadboard.kicad_sch (KiCad schematic)
At the start: 0 parts

Commit message: Rebuild KiCad schematic as proper wiring diagram with component blocks
Replaced text-only pin list with actual visual diagram: component boxes
(rectangles) for Pico WH, GPS, joystick, e-Paper, HC-SR04, and speaker
connected by polyline wires. Includes voltage divider detail, speaker
transistor circuit, 3V3 power rail, and notes section. A2 paper size.

Co-Authored-By: Claude Opus 4.6 (1M context) <noreply@anthropic.com>
Other:
- note added: "1. HC-SR04 ECHO outputs 5V - MUST use 1K+2K voltage divider or Pico GPIO will be damaged"
- note added: "2. GPS TX connects to Pico RX (GP1), GPS RX connects to Pico TX (GP0) - crossover"
- note added: "3. HC-SR04 VCC must be 5V (VBUS pin 40), not 3.3V - sensor will not work on 3.3V"
- note added: "3V3 --> Spkr(+) --> Spkr(-) --> Collector"
- note added: "3V3 POWER RAIL (Pin 36, 300mA max)"
- note added: "4. 16 GPIO used, 10 free (GP7, GP17-22, GP26-28). Total power draw ~120mA on 300mA rail"
- note added: "5V POWER - VOLTAGE DIVIDER ON ECHO"
- note added: "Active LOW, internal pull-ups"
- note added: "CLK ----> GP10 [Pin 14]"
- note added: "COM ----> GND [Pin 8]"
- note added: "CS ----> GP9 [Pin 12]"
- note added: "DIN ----> GP11 [Pin 15]"
- note added: "DOLLATEK 5-WAY JOYSTICK"
- note added: "ECHO (5V!) --[1K]--+-- GP16 [Pin 21]"
- note added: "GND ----> GND [Pin 23]"
- note added: "GND ----> GND [Pin 3]"
- note added: "GND --> Emitter"
- note added: "GND [13]"
- note added: "GND [18]"
- note added: "GND [3]"
- note added: "GND [8] Joystick GND"
- note added: "GND [Pin 23] --> Piezo(-)"
- note added: "GP0 [1] UART0 TX"
- note added: "GP1 [2] UART0 RX"
- note added: "GP10 [14] e-Paper CLK"
- note added: "GP11 [15] e-Paper DIN"
- note added: "GP12 [16] e-Paper RST"
- note added: "GP13 [17] e-Paper BUSY"
- note added: "GP14 [19] HC-SR04 TRIG"
- note added: "GP15 PWM output"
- note added: "GP15 [20] Speaker PWM"
- note added: "GP2 [4] Joystick UP"
- note added: "GP3 [5] Joystick DOWN"
- note added: "GP4 [6] Joystick LEFT"
- note added: "GP5 [7] Joystick RIGHT"
- note added: "GP6 [9] Joystick CENTER"
- note added: "GP7 [10] FREE"
- note added: "GP8 [11] e-Paper DC"
- note added: "GP9 [12] e-Paper CS"
- note added: "GY-NEO6MV2 GPS MODULE"
- note added: "HC-SR04 ULTRASONIC"
- note added: "LOUD: GP15 --[1K]--> NPN Base"
- note added: "RASPBERRY PI PICO WH"
- note added: "RX <---- GP0 TX [Pin 1]"
- note added: "SIMPLE: GP15 [Pin 20] --> Piezo(+)"
- note added: "SPEAKER / PIEZO BUZZER"
- note added: "SPI1, 4MHz, 250x122px"
- note added: "Supplies: e-Paper VCC, GPS VCC"
- note added: "TRIG <---- GP14 [Pin 19]"
- note added: "TX ----> GP1 RX [Pin 2]"
- note added: "UART 9600 baud"
- note added: "VCC ----> 3V3 [Pin 36]"
- note added: "VCC <---- VBUS 5V [Pin 40]"
- note added: "Vout = 5 x 2K/(1K+2K) = 3.33V"
- note added: "WAVESHARE 2.13" e-PAPER V3"
- note added: "[21] GP16"
- note added: "[23] GND"
- note added: "[2K]"
- note added: "[36] 3V3 OUT"
- note added: "[37] 3V3_EN"
- note added: "[38] GND"
- note added: "[39] VSYS"
- note added: "[40] VBUS 5V"
- note removed: "1. HC-SR04 ECHO is 5V output — MUST use voltage divider or damage Pico"
- note removed: "2. GPS TX/RX crossover: GPS TX goes to Pico RX, GPS RX to Pico TX"
- note removed: "3. Joystick uses Pico internal pull-ups — no external resistors"
- note removed: "3V3 --> Speaker(+) --> Speaker(-) --> NPN Collector"
- note removed: "3V3 [Pin 36] — e-Paper VCC + GPS VCC (3.3V power)"
- note removed: "4. Speaker: piezo direct to GP15+GND, or NPN transistor for volume"
- note removed: "5. Total GPIO used: 16 of 26 — 10 pins free for future sensors"
- note removed: "6. 3V3 rail max 300mA — all peripherals draw about 120mA total"
- note removed: "CLK ----> GP10 SPI1 SCK [Pin 14]"
- note removed: "COM/GND ----> GND [Pin 8]"
- note removed: "CS ----> GP9 SPI1 CSn [Pin 12]"
- note removed: "DIN ----> GP11 SPI1 TX [Pin 15]"
- note removed: "E-PAPER DISPLAY — Waveshare 2.13 inch V3 (SPI1, 4MHz)"
- note removed: "GND ----> GND [Pin 38]"
- note removed: "GND --> NPN Emitter"
- note removed: "GND [Pin 13]"
- note removed: "GND [Pin 18]"
- note removed: "GND [Pin 23] — HC-SR04 GND + Speaker GND"
- note removed: "GND [Pin 28]"
- note removed: "GND [Pin 38] — e-Paper GND"
- note removed: "GND [Pin 3] — GPS GND"
- note removed: "GND [Pin 8] — Joystick COM / GND"
- note removed: "GP0 [Pin 1] — UART0 TX --> GPS RX"
- note removed: "GP1 [Pin 2] — UART0 RX <-- GPS TX"
- note removed: "GP10 [Pin 14] — e-Paper CLK (SPI1 SCK)"
- note removed: "GP11 [Pin 15] — e-Paper DIN (SPI1 TX / MOSI)"
- note removed: "GP12 [Pin 16] — e-Paper RST"
- note removed: "GP13 [Pin 17] — e-Paper BUSY"
- note removed: "GP14 [Pin 19] — HC-SR04 TRIG (output)"
- note removed: "GP15 [Pin 20] — Speaker PWM (output)"
- note removed: "GP16 [Pin 21] — HC-SR04 ECHO (via voltage divider)"
- note removed: "GP2 [Pin 4] — Joystick UP (pull-up, active LOW)"
- note removed: "GP3 [Pin 5] — Joystick DOWN"
- note removed: "GP4 [Pin 6] — Joystick LEFT"
- note removed: "GP5 [Pin 7] — Joystick RIGHT"
- note removed: "GP6 [Pin 9] — Joystick CENTER / SELECT"
- note removed: "GP7 [Pin 10] — FREE"
- note removed: "GP8 [Pin 11] — e-Paper DC"
- note removed: "GP9 [Pin 12] — e-Paper CS (SPI1 CSn)"
- note removed: "GPS GND ----> GND [Pin 3]"
- note removed: "GPS MODULE — GY-NEO6MV2 (UART0, 9600 baud)"
- note removed: "GPS RX <---- Pico GP0 (UART0 TX) [Pin 1] << TX-RX CROSSOVER"
- note removed: "GPS TX ----> Pico GP1 (UART0 RX) [Pin 2] << TX-RX CROSSOVER"
- note removed: "GPS VCC ----> 3V3(OUT) [Pin 36]"
- note removed: "HC-SR04 ECHO VOLTAGE DIVIDER (5V to 3.3V) — REQUIRED"
- note removed: "HC-SR04 ECHO pin ---[ 1K ohm R1 ]---+--- GP16 (Pin 21)"
- note removed: "JOYSTICK — DollaTek 5-Way (Active LOW, Internal Pull-ups)"
- note removed: "LEFT SIDE"
- note removed: "NPN transistor: 2N2222, BC547, or BC817"
- note removed: "Option A (simple): GP15 ----> Piezo(+) Piezo(-) ----> GND"
- note removed: "Option B (louder): GP15 --[ 1K R3 ]--> NPN Base"
- note removed: "RASPBERRY PI PICO WH — PIN ASSIGNMENTS"
- note removed: "RIGHT SIDE"
- note removed: "SPEAKER CIRCUIT (GP15 PWM)"
- note removed: "VBUS [Pin 40] — HC-SR04 VCC (5V)"
- note removed: "VCC ----> 3V3(OUT) [Pin 36]"
- note removed: "VSYS [Pin 39] — (Battery future)"
- note removed: "Vout = 5V x 2K / (1K + 2K) = 3.33V -- Safe for Pico 3.3V GPIO"
- note removed: "[ 2K ohm R2 ]"
- company: Dilder Project — github.com/rompasaurus/dilder -> github.com/rompasaurus/dilder
- title: Dilder Breadboard Test Bench — Full Wiring Reference -> Dilder Breadboard Wiring Diagram
