File: hardware-design/kicad/dilder-breadboard/dilder-breadboard.kicad_sch (KiCad schematic)
At the start: 0 parts

Commit message: Rebuild KiCad schematic v1.2 — fix layout, alignment, and wire routing
Rebuilt from scratch with consistent 10mm pin spacing, properly aligned
wire endpoints matching pin Y-coordinates, component boxes with clear
labels, voltage divider detail inside HC-SR04 box, and warnings section.

Co-Authored-By: Claude Opus 4.6 (1M context) <noreply@anthropic.com>
Other:
- note added: "1. HC-SR04 ECHO is 5V! Use 1K+2K divider or Pico GPIO dies"
- note added: "2. GPS TX->Pico RX (GP1), GPS RX<-Pico TX (GP0) CROSSOVER"
- note added: "3. HC-SR04 needs 5V on VBUS [40], will not work on 3.3V"
- note added: "3V3 OUT [36]"
- note added: "3V3->Spkr+->Spkr-->Collector"
- note added: "4. GPIO used: 16/26. Free: GP7,GP17-22,GP26-28"
- note added: "5V power! Divider on ECHO!"
- note added: "Active LOW Pull-ups"
- note added: "BUSY -> GP13 [17]"
- note added: "CENTER -> GP6 [9]"
- note added: "CLK -> GP10 [14]"
- note added: "COM -> GND [8]"
- note added: "CS -> GP9 [12]"
- note added: "DC -> GP8 [11]"
- note added: "DILDER BREADBOARD WIRING DIAGRAM"
- note added: "DIN -> GP11 [15]"
- note added: "DOWN -> GP3 [5]"
- note added: "ECHO 5V out:"
- note added: "ECHO--[1K]--+--GP16 [21]"
- note added: "GND -> Emitter"
- note added: "GND -> GND [23]"
- note added: "GND [23]"
- note added: "GND [38]"
- note added: "GND [8]"
- note added: "GP0 [1]"
- note added: "GP1 [2]"
- note added: "GP10 [14]"
- note added: "GP11 [15]"
- note added: "GP12 [16]"
- note added: "GP13 [17]"
- note added: "GP14 [19]"
- note added: "GP15 [20]"
- note added: "GP16 [21]"
- note added: "GP2 [4]"
- note added: "GP3 [5]"
- note added: "GP4 [6]"
- note added: "GP5 [7]"
- note added: "GP6 [9]"
- note added: "GP8 [11]"
- note added: "GP9 [12]"
- note added: "GPS GY-NEO6MV2"
- note added: "HC-SR04 uses VBUS 5V separately."
- note added: "JOYSTICK 5-Way"
- note added: "LEFT -> GP4 [6]"
- note added: "Loud: GP15-[1K]->NPN Base"
- note added: "Max 300mA. Drawing ~120mA total."
- note added: "PICO WH"
- note added: "POWER RAIL 3V3 [Pin 36]"
- note added: "PWM on GP15 [20]"
- note added: "RIGHT -> GP5 [7]"
- note added: "RST -> GP12 [16]"
- note added: "RX <--- GP0 TX [1]"
- note added: "SPEAKER / BUZZER"
- note added: "SPI1 4MHz 250x122"
- note added: "Simple: GP15 -> Piezo+ -> Piezo- -> GND"
- note added: "Supplies: e-Paper VCC + GPS VCC"
- note added: "TRIG <- GP14 [19]"
- note added: "TX ---> GP1 RX [2]"
- note added: "UART0 9600 baud"
- note added: "UP -> GP2 [4]"
- note added: "VBUS 5V [40]"
- note added: "VCC -> 3V3 GND -> GND[3]"
- note added: "VCC <- VBUS 5V [40]"
- note added: "WARNINGS"
- note added: "e-PAPER 2.13in V3"
- note removed: "1. HC-SR04 ECHO outputs 5V - MUST use 1K+2K voltage divider or Pico GPIO will be damaged"
- note removed: "2. GPS TX connects to Pico RX (GP1), GPS RX connects to Pico TX (GP0) - crossover"
- note removed: "3. HC-SR04 VCC must be 5V (VBUS pin 40), not 3.3V - sensor will not work on 3.3V"
- note removed: "3V3 --> Spkr(+) --> Spkr(-) --> Collector"
- note removed: "3V3 POWER RAIL (Pin 36, 300mA max)"
- note removed: "4. 16 GPIO used, 10 free (GP7, GP17-22, GP26-28). Total power draw ~120mA on 300mA rail"
- note removed: "5V POWER - VOLTAGE DIVIDER ON ECHO"
- note removed: "Active LOW, internal pull-ups"
- note removed: "BUSY ----> GP13 [Pin 17]"
- note removed: "CENTER ----> GP6 [Pin 9]"
- note removed: "CLK ----> GP10 [Pin 14]"
- note removed: "COM ----> GND [Pin 8]"
- note removed: "CS ----> GP9 [Pin 12]"
- note removed: "DC ----> GP8 [Pin 11]"
- note removed: "DIN ----> GP11 [Pin 15]"
- note removed: "DOLLATEK 5-WAY JOYSTICK"
- note removed: "DOWN ----> GP3 [Pin 5]"
- note removed: "ECHO (5V!) --[1K]--+-- GP16 [Pin 21]"
- note removed: "GND ----> GND [Pin 23]"
- note removed: "GND ----> GND [Pin 3]"
- note removed: "GND --> Emitter"
- note removed: "GND [13]"
- note removed: "GND [18]"
- note removed: "GND [8] Joystick GND"
- note removed: "GND [Pin 23] --> Piezo(-)"
- note removed: "GP0 [1] UART0 TX"
- note removed: "GP1 [2] UART0 RX"
- note removed: "GP10 [14] e-Paper CLK"
- note removed: "GP11 [15] e-Paper DIN"
- note removed: "GP12 [16] e-Paper RST"
- note removed: "GP13 [17] e-Paper BUSY"
- note removed: "GP14 [19] HC-SR04 TRIG"
- note removed: "GP15 PWM output"
- note removed: "GP15 [20] Speaker PWM"
- note removed: "GP2 [4] Joystick UP"
- note removed: "GP3 [5] Joystick DOWN"
- note removed: "GP4 [6] Joystick LEFT"
- note removed: "GP5 [7] Joystick RIGHT"
- note removed: "GP6 [9] Joystick CENTER"
- note removed: "GP7 [10] FREE"
- note removed: "GP8 [11] e-Paper DC"
- note removed: "GP9 [12] e-Paper CS"
- note removed: "GY-NEO6MV2 GPS MODULE"
- note removed: "LEFT ----> GP4 [Pin 6]"
- note removed: "LOUD: GP15 --[1K]--> NPN Base"
- note removed: "NOTES"
- note removed: "RASPBERRY PI PICO WH"
- note removed: "RIGHT ----> GP5 [Pin 7]"
- note removed: "RST ----> GP12 [Pin 16]"
- note removed: "RX <---- GP0 TX [Pin 1]"
- note removed: "SIMPLE: GP15 [Pin 20] --> Piezo(+)"
- note removed: "SPEAKER / PIEZO BUZZER"
- note removed: "SPI1, 4MHz, 250x122px"
- note removed: "Supplies: e-Paper VCC, GPS VCC"
- note removed: "TRIG <---- GP14 [Pin 19]"
- note removed: "TX ----> GP1 RX [Pin 2]"
- note removed: "UART 9600 baud"
- note removed: "UP ----> GP2 [Pin 4]"
- note removed: "VCC ----> 3V3 [Pin 36]"
- note removed: "VCC <---- VBUS 5V [Pin 40]"
- note removed: "Vout = 5 x 2K/(1K+2K) = 3.33V"
- note removed: "WAVESHARE 2.13" e-PAPER V3"
- note removed: "[21] GP16"
- note removed: "[23] GND"
- note removed: "[36] 3V3 OUT"
- note removed: "[37] 3V3_EN"
- note removed: "[38] GND"
- note removed: "[39] VSYS"
- note removed: "[40] VBUS 5V"
