File: hardware-design/PCB Designs/Dilder Full Board/Dilder-Full-board/Dilder-Full-board.kicad_sch (KiCad schematic)
At the start: 0 parts

Commit message: copied in a few component schematics to the full board
Parts:
- added +3V3: +3V3, TestPoint:TestPoint_Pad_D1.0mm, symbol Connector:TestPoint
- added A1: RaspberryPi_Pico_W, Module:RaspberryPi_Pico_W_SMD, symbol MCU_Module:RaspberryPi_Pico_W_Extensive
- added C2, C20, C36, C6, C7, C8: 10uF, Capacitor_SMD:C_0402_1005Metric, symbol Device:C
- added C22, C35: 0.1uF, Capacitor_SMD:C_0402_1005Metric, symbol Device:C
- added C29, C30, C34, C41: 1uF, Capacitor_SMD:C_0603_1608Metric, symbol Device:C
- added C48, C49, C50, C51, C52, C53, C54, C55: 4.7uF, Capacitor_SMD:C_0805_2012Metric, symbol Device:C
- added D1: LED, LED_SMD:LED_0603_1608Metric, symbol Device:LED
- added D4, D5, D6, D7: SS14, Diode_SMD:D_SMA, symbol Diode:SS14
- added J1: USB_C_Receptacle_USB2.0_14P, Connector_USB:USB_C_Receptacle_HCTL_HC-TYPE-C-16P-01A, symbol Connector:USB_C_Receptacle_USB2.0_14P
- added J2: Conn_01x02_Pin, Connector_PinSocket_2.54mm:PinSocket_1x02_P2.54mm_Vertical, symbol Connector:Conn_01x02_Pin
- added JP1: SolderJumper_3_Bridged12, Jumper:SolderJumper-3_P1.3mm_Bridged12_RoundedPad1.0x1.5mm_NumberLabels, symbol Jumper:SolderJumper_3_Bridged12
- added L4: 10uH, Inductor_SMD:L_Ferrocore_DLG-0403, symbol Device:L
- added P4: AFC07-S24FCC-00, Connector_FFC-FPC:Jushuo_AFC07-S24FCA-00_1x24-1MP_P0.50_Horizontal, symbol 03_EINK-SchDoc-rescue:SFV24R-1STE1HLF-
- added Q1: AO3401A, Package_TO_SOT_SMD:SOT-23, symbol Transistor_FET:AO3401A
- added Q3: AO3400A, Package_TO_SOT_SMD:SOT-23, symbol Transistor_FET:AO3400A
- added R1: 2K, Resistor_SMD:R_0402_1005Metric, symbol Device:R
- added R12, R19: 200K, Resistor_SMD:R_0402_1005Metric, symbol Device:R
- added R14, R17: 5.1K, Resistor_SMD:R_0402_1005Metric, symbol Device:R
- added R18, R2: 33R, Resistor_SMD:R_0402_1005Metric, symbol Device:R
- added R20: 100K, Resistor_SMD:R_0402_1005Metric, symbol Device:R
- added R3, R33, R35: 10K, Resistor_SMD:R_0402_1005Metric, symbol Device:R
- added R34, R37: 2.2R, Resistor_SMD:R_0603_1608Metric, symbol Device:R
- added R36, R38: 1R, Resistor_SMD:R_0603_1608Metric, symbol Device:R
- added U2: W25Q128JVS, Package_SO:SOIC-8_5.3x5.3mm_P1.27mm, symbol Memory_Flash:W25Q128JVS
- added U3: MCP73831-2-OT, Package_TO_SOT_SMD:SOT-23-5, symbol Battery_Management:MCP73831-2-OT
- added U4: AMS1117-3.3, Package_TO_SOT_SMD:SOT-223-3_TabPin2, symbol Regulator_Linear:AMS1117-3.3
Connections:
- new net: C30.1, P4.18 (VDD)
- new net: C29.1, P4.19 (VPP)
- new net: C55.1, P4.20 (VSH1)
- new net: C54.1, P4.22 (VSL)
- new net: C52.1, P4.4 (NC)
- new net: C53.1, P4.5 (VSH2)
- new net: P4.8 (BS1), R33.1, R37.2
- new net: C49.1, D5.2 (A), D6.1 (K)
- new net: C49.2, D7.2 (A), L4.2, Q3.3 (D)
- new net: J1.A5 (CC1), R14.2
- new net: J1.B5 (CC2), R17.2
- new net: JP1.3 (B), R36.2, R38.2
- new net: D1.1 (K), R3.2
- new net: JP1.1 (A), R34.2
- new net: R3.1, U3.1 (STAT)
- new net: R1.2, U3.5 (PROG)
- new net: A1.13 (GND), A1.18 (GND), A1.23 (GND), A1.28 (GND), A1.3 (GND), A1.38 (GND), A1.8 (GND), A1.D2 (GND)
- new net: JP1.2 (C), Q3.2 (S)
- new net +3V3: +3V3.1, C20.1, C35.1, C41.1, C51.1, L4.1, P4.15 (VDDIO), P4.16 (VCI), U4.2 (VO)
- new net 5V: C22.1, C36.1, C6.1, D1.2 (A), D4.2 (A), J1.A4 (VBUS), J1.A9 (VBUS), J1.B4 (VBUS), J1.B9 (VBUS), Q1.1 (G), R20.2, U3.4 (V_{DD})
- new net GDR: P4.2 (GDR), Q3.1 (G), R35.2
- new net GND: C2.2, C20.2, C22.2, C29.2, C30.2, C34.2, C35.2, C36.2, C41.2, C48.2, C50.2, C51.2, C52.2, C53.2, C54.2, C55.2, C6.2, C7.2, C8.2, D5.1 (K), J1.A1 (GND), J1.A12 (GND), J1.B1 (GND), J1.B12 (GND), J1.S1 (SHIELD), J2.1 (Pin_1), P4.17 (VSS), R1.1, R14.1, R17.1, R19.2, R20.1, R34.1, R35.1, R36.1, R37.1, R38.1, U2.4 (GND), U3.2 (V_{SS}), U4.1 (GND)
- new net IO17_DISP_nCS: P4.12 (~{CS})
- new net IO18_DISP_SCL: P4.13 (SCL)
- new net IO21_DISP_SDA: P4.14 (SDA)
- new net IO33_DISP_BUSY: P4.9 (BUSY)
- new net IO34_DISP_RESET: P4.10 (RESET)
- new net IO48_DISP_DATA/nCMD: P4.11 (DATA/~{CM}D)
- new net IO4/BAT: R12.2, R19.1
- new net PREVGH: C50.1, D7.1 (K), P4.21 (VGH)
- new net PREVGL: C48.1, D6.2 (A), P4.23 (VGL)
- new net RESE: P4.3 (RSENSE)
- new net SPICS0: U2.1 (~{CS})
- new net SPID: U2.5 (DI/IO_{0})
- new net SPIHD: U2.7 (~{HOLD}/~{RESET}/IO_{3})
- new net SPIQ: U2.2 (DO/IO_{1})
- new net SPISCK: U2.6 (CLK)
- new net SPIWP: U2.3 (~{WP}/IO_{2})
- new net USB_D+: J1.A6 (D+), J1.B6 (D+), R18.1, R18.2
- new net USB_D-: J1.A7 (D-), J1.B7 (D-), R2.1, R2.2
- new net VBAT: C2.1, C8.1, J2.2 (Pin_2), Q1.3 (D), R12.1, U3.3 (V_{BAT})
- new net VCOM: C34.1, P4.24 (VCOM)
- new net VDD_CPU: R33.2
- new net VDD_SPI: U2.8 (VCC)
- new net VSYS: C7.1, D4.1 (K), Q1.2 (S), U4.3 (VI)
- no-connect marks 0 -> 3
Other:
- note added: "BATTERY CHARGER"
- note added: "MEMORY"
- note added: "USB-C"
- note added: "VOLTAGE REGULATOR"
- title: (none) -> Dilder Full Board Accel Chargin Joystick display and Sound
